Commit message: feat: rename rover_description into xplore_description

File: xplore_description/urdf/assemblage.urdf.xacro (robot description, xacro)
@@ -1,12 +1,12 @@
 <?xml version="1.0" ?>
 <robot name="kerby" xmlns:xacro="http://www.ros.org/wiki/xacro">
-<xacro:include filename="$(find rover_description)/urdf/materials.xacro" />
-<xacro:include filename="$(find rover_description)/urdf/kerby.trans" />
-<xacro:include filename="$(find rover_description)/urdf/kerby.gazebo" />
-<xacro:include filename="$(find rover_description)/urdf/ouster.xacro" />
-<xacro:include filename="$(find rover_description)/urdf/imu.xacro" />
-<xacro:include filename="$(find rover_description)/urdf/inertial_macros.xacro" />
-<xacro:include filename="$(find rover_description)/urdf/oakd_camera.xacro" />
-<xacro:include filename="$(find rover_description)/urdf/ros2_control.xacro" />
+<xacro:include filename="$(find xplore_description)/urdf/materials.xacro" />
+<xacro:include filename="$(find xplore_description)/urdf/kerby.trans" />
+<xacro:include filename="$(find xplore_description)/urdf/kerby.gazebo" />
+<xacro:include filename="$(find xplore_description)/urdf/ouster.xacro" />
+<xacro:include filename="$(find xplore_description)/urdf/imu.xacro" />
+<xacro:include filename="$(find xplore_description)/urdf/inertial_macros.xacro" />
+<xacro:include filename="$(find xplore_description)/urdf/oakd_camera.xacro" />
+<xacro:include filename="$(find xplore_description)/urdf/ros2_control.xacro" />
 <xacro:property name="rpm_to_Radps" value="${2*pi/60.0}" />     <!-- rotations per minute to Rad per second conversion -->
 <xacro:property name="velocity_scaling" value="1.0" />     <!-- allows to scale all max velocities down at once -->
@@ -48,5 +48,5 @@
     <origin xyz="0 0 0" rpy="0 0 0"/>
     <geometry>
-      <mesh filename="file://$(find rover_description)/meshes/base_link.stl" scale="0.001 0.001 0.001"/>
+      <mesh filename="file://$(find xplore_description)/meshes/base_link.stl" scale="0.001 0.001 0.001"/>
     </geometry>
     <material name="blue"/>
@@ -55,5 +55,5 @@
     <origin xyz="0 0 0" rpy="0 0 0"/>
     <geometry>
-      <mesh filename="file://$(find rover_description)/meshes/base_link.stl" scale="0.001 0.001 0.001"/>
+      <mesh filename="file://$(find xplore_description)/meshes/base_link.stl" scale="0.001 0.001 0.001"/>
     </geometry>
   </collision>
@@ -68,5 +68,5 @@
     <origin xyz="-0.421384 -0.393882 0.063562" rpy="0 0 0"/>
     <geometry>
-      <mesh filename="file://$(find rover_description)/meshes/steering_1.stl" scale="0.001 0.001 0.001"/>
+      <mesh filename="file://$(find xplore_description)/meshes/steering_1.stl" scale="0.001 0.001 0.001"/>
     </geometry>
     <material name="silver"/>
@@ -75,5 +75,5 @@
     <origin xyz="-0.421384 -0.393882 0.063562" rpy="0 0 0"/>
     <geometry>
-      <mesh filename="file://$(find rover_description)/meshes/steering_1.stl" scale="0.001 0.001 0.001"/>
+      <mesh filename="file://$(find xplore_description)/meshes/steering_1.stl" scale="0.001 0.001 0.001"/>
     </geometry>
   </collision>
@@ -88,5 +88,5 @@
     <origin xyz="-0.42341 0.353934 0.012408" rpy="0 0 0"/>
     <geometry>
-      <mesh filename="file://$(find rover_description)/meshes/steering_2.stl" scale="0.001 0.001 0.001"/>
+      <mesh filename="file://$(find xplore_description)/meshes/steering_2.stl" scale="0.001 0.001 0.001"/>
     </geometry>
     <material name="silver"/>
@@ -95,5 +95,5 @@
     <origin xyz="-0.42341 0.353934 0.012408" rpy="0 0 0"/>
     <geometry>
-      <mesh filename="file://$(find rover_description)/meshes/steering_2.stl" scale="0.001 0.001 0.001"/>
+      <mesh filename="file://$(find xplore_description)/meshes/steering_2.stl" scale="0.001 0.001 0.001"/>
     </geometry>
   </collision>
@@ -108,5 +108,5 @@
     <origin xyz="0.408171 0.353934 0.063562" rpy="0 0 0"/>
     <geometry>
-      <mesh filename="file://$(find rover_description)/meshes/steering_3.stl" scale="0.001 0.001 0.001"/>
+      <mesh filename="file://$(find xplore_description)/meshes/steering_3.stl" scale="0.001 0.001 0.001"/>
     </geometry>
     <material name="silver"/>
@@ -115,5 +115,5 @@
     <origin xyz="0.408171 0.353934 0.063562" rpy="0 0 0"/>
     <geometry>
-      <mesh filename="file://$(find rover_description)/meshes/steering_3.stl" scale="0.001 0.001 0.001"/>
+      <mesh filename="file://$(find xplore_description)/meshes/steering_3.stl" scale="0.001 0.001 0.001"/>
     </geometry>
   </collision>
@@ -128,5 +128,5 @@
     <origin xyz="0.410197 -0.393882 0.012408" rpy="0 0 0"/>
     <geometry>
-      <mesh filename="file://$(find rover_description)/meshes/steering_4.stl" scale="0.001 0.001 0.001"/>
+      <mesh filename="file://$(find xplore_description)/meshes/steering_4.stl" scale="0.001 0.001 0.001"/>
     </geometry>
     <material name="silver"/>
@@ -135,5 +135,5 @@
     <origin xyz="0.410197 -0.393882 0.012408" rpy="0 0 0"/>
     <geometry>
-      <mesh filename="file://$(find rover_description)/meshes/steering_4.stl" scale="0.001 0.001 0.001"/>
+      <mesh filename="file://$(find xplore_description)/meshes/steering_4.stl" scale="0.001 0.001 0.001"/>
     </geometry>
   </collision>
@@ -148,5 +148,5 @@
     <origin xyz="0.42733 -0.410572 0.281864" rpy="0 0 0"/>
     <geometry>
-      <mesh filename="file://$(find rover_description)/meshes/wheel3_1.stl" scale="0.001 0.001 0.001"/>
+      <mesh filename="file://$(find xplore_description)/meshes/wheel3_1.stl" scale="0.001 0.001 0.001"/>
     </geometry>
     <material name="pink"/>
@@ -155,5 +155,5 @@
     <origin xyz="0.42733 -0.410572 0.281864" rpy="0 0 0"/>
     <geometry>
-      <mesh filename="file://$(find rover_description)/meshes/wheel3_1.stl" scale="0.001 0.001 0.001"/>
+      <mesh filename="file://$(find xplore_description)/meshes/wheel3_1.stl" scale="0.001 0.001 0.001"/>
     </geometry>
   </collision>
@@ -168,5 +168,5 @@
     <origin xyz="-0.404251 -0.410572 0.333019" rpy="0 0 0"/>
     <geometry>
-      <mesh filename="file://$(find rover_description)/meshes/wheel4_1.stl" scale="0.001 0.001 0.001"/>
+      <mesh filename="file://$(find xplore_description)/meshes/wheel4_1.stl" scale="0.001 0.001 0.001"/>
     </geometry>
     <material name="pink"/>
@@ -175,5 +175,5 @@
     <origin xyz="-0.404251 -0.410572 0.333019" rpy="0 0 0"/>
     <geometry>
-      <mesh filename="file://$(find rover_description)/meshes/wheel4_1.stl" scale="0.001 0.001 0.001"/>
+      <mesh filename="file://$(find xplore_description)/meshes/wheel4_1.stl" scale="0.001 0.001 0.001"/>
     </geometry>
   </collision>
@@ -188,5 +188,5 @@
     <origin xyz="0.391037 0.370625 0.333019" rpy="0 0 0"/>
     <geometry>
-      <mesh filename="file://$(find rover_description)/meshes/wheel2_1.stl" scale="0.001 0.001 0.001"/>
+      <mesh filename="file://$(find xplore_description)/meshes/wheel2_1.stl" scale="0.001 0.001 0.001"/>
     </geometry>
     <material name="pink"/>
@@ -195,5 +195,5 @@
     <origin xyz="0.391037 0.370625 0.333019" rpy="0 0 0"/>
     <geometry>
-      <mesh filename="file://$(find rover_description)/meshes/wheel2_1.stl" scale="0.001 0.001 0.001"/>
+      <mesh filename="file://$(find xplore_description)/meshes/wheel2_1.stl" scale="0.001 0.001 0.001"/>
     </geometry>
   </collision>
@@ -208,5 +208,5 @@
     <origin xyz="-0.440543 0.370625 0.281864" rpy="0 0 0"/>
     <geometry>
-      <mesh filename="file://$(find rover_description)/meshes/wheel1_1.stl" scale="0.001 0.001 0.001"/>
+      <mesh filename="file://$(find xplore_description)/meshes/wheel1_1.stl" scale="0.001 0.001 0.001"/>
     </geometry>
     <material name="pink"/>
@@ -215,5 +215,5 @@
     <origin xyz="-0.440543 0.370625 0.281864" rpy="0 0 0"/>
     <geometry>
-      <mesh filename="file://$(find rover_description)/meshes/wheel1_1.stl" scale="0.001 0.001 0.001"/>
+      <mesh filename="file://$(find xplore_description)/meshes/wheel1_1.stl" scale="0.001 0.001 0.001"/>
     </geometry>
   </collision>
@@ -228,5 +228,5 @@
     <origin xyz="-0.006607 -0.250474 0.021516" rpy="0 0 0"/>
     <geometry>
-      <mesh filename="file://$(find rover_description)/meshes/pivot_droit_1.stl" scale="0.001 0.001 0.001"/>
+      <mesh filename="file://$(find xplore_description)/meshes/pivot_droit_1.stl" scale="0.001 0.001 0.001"/>
     </geometry>
     <material name="black"/>
@@ -235,5 +235,5 @@
     <origin xyz="-0.006607 -0.250474 0.021516" rpy="0 0 0"/>
     <geometry>
-      <mesh filename="file://$(find rover_description)/meshes/pivot_droit_1.stl" scale="0.001 0.001 0.001"/>
+      <mesh filename="file://$(find xplore_description)/meshes/pivot_droit_1.stl" scale="0.001 0.001 0.001"/>
     </geometry>
   </collision>
@@ -248,5 +248,5 @@
     <origin xyz="-0.006607 0.210526 0.021516" rpy="0 0 0"/>
     <geometry>
-      <mesh filename="file://$(find rover_description)/meshes/pivot_gauche_1.stl" scale="0.001 0.001 0.001"/>
+      <mesh filename="file://$(find xplore_description)/meshes/pivot_gauche_1.stl" scale="0.001 0.001 0.001"/>
     </geometry>
     <material name="black"/>
@@ -255,5 +255,5 @@
     <origin xyz="-0.006607 0.210526 0.021516" rpy="0 0 0"/>
     <geometry>
-      <mesh filename="file://$(find rover_description)/meshes/pivot_gauche_1.stl" scale="0.001 0.001 0.001"/>
+      <mesh filename="file://$(find xplore_description)/meshes/pivot_gauche_1.stl" scale="0.001 0.001 0.001"/>
     </geometry>
   </collision>

File: xplore_description/urdf/imu.xacro (robot description, xacro)
@@ -1,5 +1,5 @@
 <?xml version="1.0"?>
 <robot xmlns:xacro="http://www.ros.org/wiki/xacro" name="imu">
-<xacro:include filename="$(find rover_description)/urdf/inertial_macros.xacro" />
+<xacro:include filename="$(find xplore_description)/urdf/inertial_macros.xacro" />
     <joint name="imu_joint" type="fixed">
         <origin xyz="0.2 0 0.11" rpy="0 0 -${pi}"/>

File: xplore_description/urdf/oakd_camera.xacro (robot description, xacro)
@@ -15,5 +15,5 @@
     <visual name="camera_visual">
       <geometry>
-          <mesh filename="file://$(find rover_description)/meshes/OAK-D.dae" />
+          <mesh filename="file://$(find xplore_description)/meshes/OAK-D.dae" />
         </geometry>
     </visual>

File: xplore_description/urdf/ouster.xacro (robot description, xacro)
@@ -10,5 +10,5 @@
         <visual>
           <geometry>
-            <mesh filename="file://$(find rover_description)/meshes/os1.dae" />
+            <mesh filename="file://$(find xplore_description)/meshes/os1.dae" />
             </geometry>
         </visual>

File: xplore_description/urdf/ros2_control.xacro (robot description, xacro)
@@ -72,5 +72,5 @@
     <gazebo>
         <plugin name="gazebo_ros2_control" filename="libgazebo_ros2_control.so">
-            <parameters>$(find rover_description)/config/control.yaml</parameters>
+            <parameters>$(find xplore_description)/config/control.yaml</parameters>
         </plugin>
     </gazebo>

Commit message: feat: refactor meshes organization

File: xplore_description/urdf/assemblage.urdf.xacro (robot description, xacro)
@@ -48,5 +48,5 @@
     <origin xyz="0 0 0" rpy="0 0 0"/>
     <geometry>
-      <mesh filename="file://$(find xplore_description)/meshes/base_link.stl" scale="0.001 0.001 0.001"/>
+      <mesh filename="file://$(find xplore_description)/meshes/rover/base_link.stl" scale="0.001 0.001 0.001"/>
     </geometry>
     <material name="blue"/>
@@ -55,5 +55,5 @@
     <origin xyz="0 0 0" rpy="0 0 0"/>
     <geometry>
-      <mesh filename="file://$(find xplore_description)/meshes/base_link.stl" scale="0.001 0.001 0.001"/>
+      <mesh filename="file://$(find xplore_description)/meshes/rover/base_link.stl" scale="0.001 0.001 0.001"/>
     </geometry>
   </collision>
@@ -68,5 +68,5 @@
     <origin xyz="-0.421384 -0.393882 0.063562" rpy="0 0 0"/>
     <geometry>
-      <mesh filename="file://$(find xplore_description)/meshes/steering_1.stl" scale="0.001 0.001 0.001"/>
+      <mesh filename="file://$(find xplore_description)/meshes/rover/steering_1.stl" scale="0.001 0.001 0.001"/>
     </geometry>
     <material name="silver"/>
@@ -75,5 +75,5 @@
     <origin xyz="-0.421384 -0.393882 0.063562" rpy="0 0 0"/>
     <geometry>
-      <mesh filename="file://$(find xplore_description)/meshes/steering_1.stl" scale="0.001 0.001 0.001"/>
+      <mesh filename="file://$(find xplore_description)/meshes/rover/steering_1.stl" scale="0.001 0.001 0.001"/>
     </geometry>
   </collision>
@@ -88,5 +88,5 @@
     <origin xyz="-0.42341 0.353934 0.012408" rpy="0 0 0"/>
     <geometry>
-      <mesh filename="file://$(find xplore_description)/meshes/steering_2.stl" scale="0.001 0.001 0.001"/>
+      <mesh filename="file://$(find xplore_description)/meshes/rover/steering_2.stl" scale="0.001 0.001 0.001"/>
     </geometry>
     <material name="silver"/>
@@ -95,5 +95,5 @@
     <origin xyz="-0.42341 0.353934 0.012408" rpy="0 0 0"/>
     <geometry>
-      <mesh filename="file://$(find xplore_description)/meshes/steering_2.stl" scale="0.001 0.001 0.001"/>
+      <mesh filename="file://$(find xplore_description)/meshes/rover/steering_2.stl" scale="0.001 0.001 0.001"/>
     </geometry>
   </collision>
@@ -108,5 +108,5 @@
     <origin xyz="0.408171 0.353934 0.063562" rpy="0 0 0"/>
     <geometry>
-      <mesh filename="file://$(find xplore_description)/meshes/steering_3.stl" scale="0.001 0.001 0.001"/>
+      <mesh filename="file://$(find xplore_description)/meshes/rover/steering_3.stl" scale="0.001 0.001 0.001"/>
     </geometry>
     <material name="silver"/>
@@ -115,5 +115,5 @@
     <origin xyz="0.408171 0.353934 0.063562" rpy="0 0 0"/>
     <geometry>
-      <mesh filename="file://$(find xplore_description)/meshes/steering_3.stl" scale="0.001 0.001 0.001"/>
+      <mesh filename="file://$(find xplore_description)/meshes/rover/steering_3.stl" scale="0.001 0.001 0.001"/>
     </geometry>
   </collision>
@@ -128,5 +128,5 @@
     <origin xyz="0.410197 -0.393882 0.012408" rpy="0 0 0"/>
     <geometry>
-      <mesh filename="file://$(find xplore_description)/meshes/steering_4.stl" scale="0.001 0.001 0.001"/>
+      <mesh filename="file://$(find xplore_description)/meshes/rover/steering_4.stl" scale="0.001 0.001 0.001"/>
     </geometry>
     <material name="silver"/>
@@ -135,5 +135,5 @@
     <origin xyz="0.410197 -0.393882 0.012408" rpy="0 0 0"/>
     <geometry>
-      <mesh filename="file://$(find xplore_description)/meshes/steering_4.stl" scale="0.001 0.001 0.001"/>
+      <mesh filename="file://$(find xplore_description)/meshes/rover/steering_4.stl" scale="0.001 0.001 0.001"/>
     </geometry>
   </collision>
@@ -148,5 +148,5 @@
     <origin xyz="0.42733 -0.410572 0.281864" rpy="0 0 0"/>
     <geometry>
-      <mesh filename="file://$(find xplore_description)/meshes/wheel3_1.stl" scale="0.001 0.001 0.001"/>
+      <mesh filename="file://$(find xplore_description)/meshes/rover/wheel3_1.stl" scale="0.001 0.001 0.001"/>
     </geometry>
     <material name="pink"/>
@@ -155,5 +155,5 @@
     <origin xyz="0.42733 -0.410572 0.281864" rpy="0 0 0"/>
     <geometry>
-      <mesh filename="file://$(find xplore_description)/meshes/wheel3_1.stl" scale="0.001 0.001 0.001"/>
+      <mesh filename="file://$(find xplore_description)/meshes/rover/wheel3_1.stl" scale="0.001 0.001 0.001"/>
     </geometry>
   </collision>
@@ -168,5 +168,5 @@
     <origin xyz="-0.404251 -0.410572 0.333019" rpy="0 0 0"/>
     <geometry>
-      <mesh filename="file://$(find xplore_description)/meshes/wheel4_1.stl" scale="0.001 0.001 0.001"/>
+      <mesh filename="file://$(find xplore_description)/meshes/rover/wheel4_1.stl" scale="0.001 0.001 0.001"/>
     </geometry>
     <material name="pink"/>
@@ -175,5 +175,5 @@
     <origin xyz="-0.404251 -0.410572 0.333019" rpy="0 0 0"/>
     <geometry>
-      <mesh filename="file://$(find xplore_description)/meshes/wheel4_1.stl" scale="0.001 0.001 0.001"/>
+      <mesh filename="file://$(find xplore_description)/meshes/rover/wheel4_1.stl" scale="0.001 0.001 0.001"/>
     </geometry>
   </collision>
@@ -188,5 +188,5 @@
     <origin xyz="0.391037 0.370625 0.333019" rpy="0 0 0"/>
     <geometry>
-      <mesh filename="file://$(find xplore_description)/meshes/wheel2_1.stl" scale="0.001 0.001 0.001"/>
+      <mesh filename="file://$(find xplore_description)/meshes/rover/wheel2_1.stl" scale="0.001 0.001 0.001"/>
     </geometry>
     <material name="pink"/>
@@ -195,5 +195,5 @@
     <origin xyz="0.391037 0.370625 0.333019" rpy="0 0 0"/>
     <geometry>
-      <mesh filename="file://$(find xplore_description)/meshes/wheel2_1.stl" scale="0.001 0.001 0.001"/>
+      <mesh filename="file://$(find xplore_description)/meshes/rover/wheel2_1.stl" scale="0.001 0.001 0.001"/>
     </geometry>
   </collision>
@@ -208,5 +208,5 @@
     <origin xyz="-0.440543 0.370625 0.281864" rpy="0 0 0"/>
     <geometry>
-      <mesh filename="file://$(find xplore_description)/meshes/wheel1_1.stl" scale="0.001 0.001 0.001"/>
+      <mesh filename="file://$(find xplore_description)/meshes/rover/wheel1_1.stl" scale="0.001 0.001 0.001"/>
     </geometry>
     <material name="pink"/>
@@ -215,5 +215,5 @@
     <origin xyz="-0.440543 0.370625 0.281864" rpy="0 0 0"/>
     <geometry>
-      <mesh filename="file://$(find xplore_description)/meshes/wheel1_1.stl" scale="0.001 0.001 0.001"/>
+      <mesh filename="file://$(find xplore_description)/meshes/rover/wheel1_1.stl" scale="0.001 0.001 0.001"/>
     </geometry>
   </collision>
@@ -228,5 +228,5 @@
     <origin xyz="-0.006607 -0.250474 0.021516" rpy="0 0 0"/>
     <geometry>
-      <mesh filename="file://$(find xplore_description)/meshes/pivot_droit_1.stl" scale="0.001 0.001 0.001"/>
+      <mesh filename="file://$(find xplore_description)/meshes/rover/pivot_droit_1.stl" scale="0.001 0.001 0.001"/>
     </geometry>
     <material name="black"/>
@@ -235,5 +235,5 @@
     <origin xyz="-0.006607 -0.250474 0.021516" rpy="0 0 0"/>
     <geometry>
-      <mesh filename="file://$(find xplore_description)/meshes/pivot_droit_1.stl" scale="0.001 0.001 0.001"/>
+      <mesh filename="file://$(find xplore_description)/meshes/rover/pivot_droit_1.stl" scale="0.001 0.001 0.001"/>
     </geometry>
   </collision>
@@ -248,5 +248,5 @@
     <origin xyz="-0.006607 0.210526 0.021516" rpy="0 0 0"/>
     <geometry>
-      <mesh filename="file://$(find xplore_description)/meshes/pivot_gauche_1.stl" scale="0.001 0.001 0.001"/>
+      <mesh filename="file://$(find xplore_description)/meshes/rover/pivot_gauche_1.stl" scale="0.001 0.001 0.001"/>
     </geometry>
     <material name="black"/>
@@ -255,5 +255,5 @@
     <origin xyz="-0.006607 0.210526 0.021516" rpy="0 0 0"/>
     <geometry>
-      <mesh filename="file://$(find xplore_description)/meshes/pivot_gauche_1.stl" scale="0.001 0.001 0.001"/>
+      <mesh filename="file://$(find xplore_description)/meshes/rover/pivot_gauche_1.stl" scale="0.001 0.001 0.001"/>
     </geometry>
   </collision>

File: xplore_description/urdf/oakd_camera.xacro (robot description, xacro)
@@ -15,5 +15,5 @@
     <visual name="camera_visual">
       <geometry>
-          <mesh filename="file://$(find xplore_description)/meshes/OAK-D.dae" />
+          <mesh filename="file://$(find xplore_description)/meshes/camera/OAK-D.dae" />
         </geometry>
     </visual>

File: xplore_description/urdf/ouster.xacro (robot description, xacro)
@@ -10,5 +10,5 @@
         <visual>
           <geometry>
-            <mesh filename="file://$(find xplore_description)/meshes/os1.dae" />
+            <mesh filename="file://$(find xplore_description)/meshes/lidar/os1.dae" />
             </geometry>
         </visual>
