Commit message: feat: refactor urdf files organization

File: xplore_description/urdf/common/materials.xacro (robot description, xacro)
@@ -1,4 +1,4 @@
 <?xml version="1.0" ?>
-<robot name="kerby" xmlns:xacro="http://www.ros.org/wiki/xacro" >
+<robot name="robot" xmlns:xacro="http://www.ros.org/wiki/xacro" >
 <material name="silver">
   <color rgba="0.700 0.700 0.700 1.000"/>

File: xplore_description/urdf/rover/camera/oakd_camera.xacro (robot description, xacro)
@@ -15,5 +15,5 @@
     <visual name="camera_visual">
       <geometry>
-          <mesh filename="file://$(find xplore_description)/meshes/camera/OAK-D.dae" />
+          <mesh filename="file://$(find xplore_description)/meshes/rover/camera/OAK-D.dae" />
         </geometry>
     </visual>

File: xplore_description/urdf/rover/imu/imu.xacro (robot description, xacro)
@@ -1,5 +1,5 @@
 <?xml version="1.0"?>
 <robot xmlns:xacro="http://www.ros.org/wiki/xacro" name="imu">
-<xacro:include filename="$(find xplore_description)/urdf/inertial_macros.xacro" />
+<xacro:include filename="$(find xplore_description)/urdf/common/inertial_macro.xacro" />
     <joint name="imu_joint" type="fixed">
         <origin xyz="0.2 0 0.11" rpy="0 0 -${pi}"/>

File: xplore_description/urdf/rover/lidar/ouster.xacro (robot description, xacro)
@@ -1,5 +1,5 @@
 <?xml version="1.0"?>
 <robot xmlns:xacro="http://ros.org/wiki/xacro">
-  <xacro:include filename="inertial_macros.xacro"/>
+  <xacro:include filename="$(find xplore_description)/urdf/common/inertial_macro.xacro" />
     <joint name="lidar_joint" type="fixed">
         <origin xyz="0.0 0 0.145" rpy="0 0 ${pi}"/>
@@ -10,5 +10,5 @@
         <visual>
           <geometry>
-            <mesh filename="file://$(find xplore_description)/meshes/lidar/os1.dae" />
+            <mesh filename="file://$(find xplore_description)/meshes/rover/lidar/os1.dae" />
             </geometry>
         </visual>

File: xplore_description/urdf/rover/rover.urdf.xacro (robot description, xacro)
@@ -1,12 +1,12 @@
 <?xml version="1.0" ?>
-<robot name="kerby" xmlns:xacro="http://www.ros.org/wiki/xacro">
-<xacro:include filename="$(find xplore_description)/urdf/materials.xacro" />
-<xacro:include filename="$(find xplore_description)/urdf/kerby.trans" />
-<xacro:include filename="$(find xplore_description)/urdf/kerby.gazebo" />
-<xacro:include filename="$(find xplore_description)/urdf/ouster.xacro" />
-<xacro:include filename="$(find xplore_description)/urdf/imu.xacro" />
-<xacro:include filename="$(find xplore_description)/urdf/inertial_macros.xacro" />
-<xacro:include filename="$(find xplore_description)/urdf/oakd_camera.xacro" />
-<xacro:include filename="$(find xplore_description)/urdf/ros2_control.xacro" />
+<robot name="rover" xmlns:xacro="http://www.ros.org/wiki/xacro">
+<xacro:include filename="$(find xplore_description)/urdf/common/materials.xacro" />
+<xacro:include filename="$(find xplore_description)/urdf/rover/rover.transmission.xacro" />
+<xacro:include filename="$(find xplore_description)/urdf/rover/rover.gazebo.xacro" />
+<xacro:include filename="$(find xplore_description)/urdf/rover/lidar/ouster.xacro" />
+<xacro:include filename="$(find xplore_description)/urdf/rover/imu/imu.xacro" />
+<xacro:include filename="$(find xplore_description)/urdf/common/inertial_macro.xacro" />
+<xacro:include filename="$(find xplore_description)/urdf/rover/camera/oakd_camera.xacro" />
+<xacro:include filename="$(find xplore_description)/urdf/rover/rover.ros2_control.xacro" />
 <xacro:property name="rpm_to_Radps" value="${2*pi/60.0}" />     <!-- rotations per minute to Rad per second conversion -->
 <xacro:property name="velocity_scaling" value="1.0" />     <!-- allows to scale all max velocities down at once -->

File: xplore_description/worlds/marsyard2022.world.xacro (robot description, xacro)
@@ -34,5 +34,5 @@
       <uri>model://marsyard2022_terrain</uri>
     </include>
-    <xacro:include filename="sdf/landmark.sdf.xacro" />
+    <xacro:include filename="$(find xplore_description)/worlds/sdf/landmark.sdf.xacro" />
     <xacro:macro name="landmark_with_offset" params="id x y z yaw">
       <xacro:property name="x_offset" value="-17.003807" />
