Commit message: fix: solve simulation bug

File: xplore_description/urdf/rover/lidar/ouster.xacro (robot description, xacro)
@@ -58,5 +58,5 @@
         </sensor>
          </gazebo>
-   <gazebo reference="lidar_link">
+   <!-- <gazebo reference="lidar_link">
         <sensor name="sensor_scan" type="ray">
           <ray>
@@ -86,4 +86,4 @@
           </plugin>
         </sensor>
-      </gazebo>
+      </gazebo>    -->
 </robot>

File: xplore_description/urdf/rover/rover.urdf.xacro (robot description, xacro)
@@ -372,5 +372,5 @@
 </joint>
 <joint name="right_pivot" type="continuous">
-  <origin xyz="0 0.250474 -0.021516" rpy="0 0 0"/>
+  <origin xyz="-0.1 0.250474 -0.021516" rpy="0 0 0"/>
   <parent link="chassis_link"/>
   <child link="right_leg"/>
@@ -378,5 +378,5 @@
 </joint>
 <joint name="left_pivot" type="continuous">
-  <origin xyz="0 -0.210526 -0.021516" rpy="0 0 0"/>
+  <origin xyz="-0.1 -0.210526 -0.021516" rpy="0 0 0"/>
   <parent link="chassis_link"/>
   <child link="left_leg"/>
