Commit message: feat: add simulated odometry

File: xplore_description/urdf/rover/camera/oakd_camera.xacro (robot description, xacro)
@@ -1,20 +1,20 @@
 <?xml version="1.0"?>
 <robot xmlns:xacro="http://ros.org/wiki/xacro">
-    <joint name="camera_joint" type="fixed">
-      <origin xyz="-0.325 0.02 0" rpy="0 0 ${pi}"/>
-      <parent link="chassis_link"/>
-      <child link="camera_link"/>
-    </joint>
-    <joint name="camera_optical_joint" type="fixed">
-        <parent link="camera_link"/>
-        <child link="camera_link_optical"/>
-        <origin xyz="0 0 0" rpy="-1.57 0 -1.57"/>
-    </joint>
-    <link name="camera_link_optical"></link>
+  <joint name="camera_joint" type="fixed">
+    <origin xyz="-0.325 0.02 0" rpy="0 0 ${pi}"/>
+    <parent link="chassis_link"/>
+    <child link="camera_link"/>
+  </joint>
+  <joint name="camera_optical_joint" type="fixed">
+    <parent link="camera_link"/>
+    <child link="camera_link_optical"/>
+    <origin xyz="0 0 0" rpy="-1.57 0 -1.57"/>
+  </joint>
+  <link name="camera_link_optical"></link>
   <link name="camera_link">
     <visual name="camera_visual">
       <geometry>
-          <mesh filename="file://$(find xplore_description)/meshes/rover/camera/OAK-D.dae" />
-        </geometry>
+        <mesh filename="file://$(find xplore_description)/meshes/rover/camera/OAK-D.dae" />
+      </geometry>
     </visual>
     <collision>
@@ -30,33 +30,33 @@
   <gazebo reference="camera_link">
     <sensor name="stereo" type="depth">
-        <always_on>true</always_on>
-        <visualize>true</visualize>
-        <update_rate>10</update_rate>
-        <camera name="stereo">
-          <horizontal_fov>1.26</horizontal_fov>
-          <vertical_fov>0.86</vertical_fov>
-          <image>
-            <width>1280</width>
-            <height>720</height>
-            <format>R8G8B8</format>
-          </image>
-          <clip>
-            <near>0.7</near>
-            <far>8.0</far>
-          </clip>
-          <noise>
-            <type>gaussian</type>
-            <mean>0.0</mean>
-            <stddev>0.007</stddev>
-          </noise>
-        </camera>
-        <plugin name="depth" filename="libgazebo_ros_camera.so">
-            <camera_name>stereo</camera_name>
-            <frame_name>camera_optical_link</frame_name>
-            <hack_baseline>0.07</hack_baseline>
-            <min_depth>0.1</min_depth>
-            <max_depth>100.0</max_depth>
-        </plugin>
-      </sensor>
-    </gazebo>
+      <always_on>true</always_on>
+      <visualize>true</visualize>
+      <update_rate>10</update_rate>
+      <camera name="stereo">
+        <horizontal_fov>1.26</horizontal_fov>
+        <vertical_fov>0.86</vertical_fov>
+        <image>
+          <width>1280</width>
+          <height>720</height>
+          <format>R8G8B8</format>
+        </image>
+        <clip>
+          <near>0.7</near>
+          <far>8.0</far>
+        </clip>
+        <noise>
+          <type>gaussian</type>
+          <mean>0.0</mean>
+          <stddev>0.007</stddev>
+        </noise>
+      </camera>
+      <plugin name="depth" filename="libgazebo_ros_camera.so">
+        <camera_name>stereo</camera_name>
+        <frame_name>camera_optical_link</frame_name>
+        <hack_baseline>0.07</hack_baseline>
+        <min_depth>0.1</min_depth>
+        <max_depth>100.0</max_depth>
+      </plugin>
+    </sensor>
+  </gazebo>
 </robot>

File: xplore_description/urdf/rover/imu/imu.xacro (robot description, xacro)
@@ -1,5 +1,5 @@
 <?xml version="1.0"?>
 <robot xmlns:xacro="http://www.ros.org/wiki/xacro" name="imu">
-<xacro:include filename="$(find xplore_description)/urdf/common/inertial_macro.xacro" />
+    <xacro:include filename="$(find xplore_description)/urdf/common/inertial_macro.xacro" />
     <joint name="imu_joint" type="fixed">
         <origin xyz="0.2 0 0.11" rpy="0 0 -${pi}"/>
@@ -31,10 +31,65 @@
             <plugin name='imu_plugin' filename='libgazebo_ros_imu_sensor.so'>
                 <ros>
-                   <namespace>/ouster</namespace>
+                    <namespace>/arduino</namespace>
                     <remapping>~/out:=imu</remapping>
                 </ros>
+                <initial_orientation_as_reference>false</initial_orientation_as_reference>
                 <output_type>sensor_msgs/msg/Imu</output_type>
                 <frame_name>imu_sensor_link</frame_name>
             </plugin>
+            <imu>
+                <angular_velocity>
+                    <x>
+                        <noise type="gaussian">
+                            <mean>0.0</mean>
+                            <stddev>2e-4</stddev>
+                            <bias_mean>0.0000075</bias_mean>
+                            <bias_stddev>0.0000008</bias_stddev>
+                        </noise>
+                    </x>
+                    <y>
+                        <noise type="gaussian">
+                            <mean>0.0</mean>
+                            <stddev>2e-4</stddev>
+                            <bias_mean>0.0000075</bias_mean>
+                            <bias_stddev>0.0000008</bias_stddev>
+                        </noise>
+                    </y>
+                    <z>
+                        <noise type="gaussian">
+                            <mean>0.0</mean>
+                            <stddev>2e-4</stddev>
+                            <bias_mean>0.0000075</bias_mean>
+                            <bias_stddev>0.0000008</bias_stddev>
+                        </noise>
+                    </z>
+                </angular_velocity>
+                <linear_acceleration>
+                    <x>
+                        <noise type="gaussian">
+                            <mean>0.0</mean>
+                            <stddev>1.7e-2</stddev>
+                            <bias_mean>0.1</bias_mean>
+                            <bias_stddev>0.001</bias_stddev>
+                        </noise>
+                    </x>
+                    <y>
+                        <noise type="gaussian">
+                            <mean>0.0</mean>
+                            <stddev>1.7e-2</stddev>
+                            <bias_mean>0.1</bias_mean>
+                            <bias_stddev>0.001</bias_stddev>
+                        </noise>
+                    </y>
+                    <z>
+                        <noise type="gaussian">
+                            <mean>0.0</mean>
+                            <stddev>1.7e-2</stddev>
+                            <bias_mean>0.1</bias_mean>
+                            <bias_stddev>0.001</bias_stddev>
+                        </noise>
+                    </z>
+                </linear_acceleration>
+            </imu>
         </sensor>
     </gazebo>

File: xplore_description/urdf/rover/rover.gazebo.xacro (robot description, xacro)
@@ -1,75 +1,101 @@
 <?xml version="1.0" ?>
-<robot name="rover" xmlns:xacro="http://www.ros.org/wiki/xacro" >
-<xacro:property name="body_color" value="Gazebo/Grey" />
-<gazebo reference="chassis_link">
-  <material>${body_color}</material>
-  <mu1>0.2</mu1>
-  <mu2>0.2</mu2>
-  <gravity>true</gravity>
-</gazebo>
-<gazebo reference="steering1_link">
-  <material>${body_color}</material>
-  <mu1>0.2</mu1>
-  <mu2>0.2</mu2>
-</gazebo>
-<gazebo reference="steering2_link">
-  <material>${body_color}</material>
-  <mu1>0.2</mu1>
-  <mu2>0.2</mu2>
-</gazebo>
-<gazebo reference="steering3_link">
-  <material>${body_color}</material>
-  <mu1>0.2</mu1>
-  <mu2>0.2</mu2>
-</gazebo>
-<gazebo reference="steering4_link">
-  <material>${body_color}</material>
-  <mu1>0.2</mu1>
-  <mu2>0.2</mu2>
-</gazebo>
-<gazebo reference="wheel3_link">
-  <material>${body_color}</material>
-  <mu1>0.2</mu1>
-  <mu2>0.2</mu2>
-</gazebo>
-<gazebo reference="wheel4_link">
-  <material>${body_color}</material>
-  <mu1>0.2</mu1>
-  <mu2>0.2</mu2>
-</gazebo>
-<gazebo reference="wheel2_link">
-  <material>${body_color}</material>
-  <mu1>0.2</mu1>
-  <mu2>0.2</mu2>
-</gazebo>
-<gazebo reference="wheel1_link">
-  <material>${body_color}</material>
-  <mu1>0.2</mu1>
-  <mu2>0.2</mu2>
-</gazebo>
-<gazebo reference="caster_wheel">
-  <material>Gazebo/Grey</material>
-  <mu1>0.2</mu1>
-  <mu2>0.2</mu2>
-</gazebo>
-<gazebo reference="caster_axis">
-  <material>Gazebo/Grey</material>
-  <mu1>0.2</mu1>
-  <mu2>0.2</mu2>
-</gazebo>
+<robot name="rover"
+  xmlns:xacro="http://www.ros.org/wiki/xacro">
+  <xacro:property name="body_color" value="Gazebo/Grey" />
+  <gazebo reference="chassis_link">
+    <material>${body_color}</material>
+    <mu1>0.2</mu1>
+    <mu2>0.2</mu2>
+    <gravity>true</gravity>
+  </gazebo>
+  <gazebo reference="steering1_link">
+    <material>${body_color}</material>
+    <mu1>0.2</mu1>
+    <mu2>0.2</mu2>
+  </gazebo>
+  <gazebo reference="steering2_link">
+    <material>${body_color}</material>
+    <mu1>0.2</mu1>
+    <mu2>0.2</mu2>
+  </gazebo>
+  <gazebo reference="steering3_link">
+    <material>${body_color}</material>
+    <mu1>0.2</mu1>
+    <mu2>0.2</mu2>
+  </gazebo>
+  <gazebo reference="steering4_link">
+    <material>${body_color}</material>
+    <mu1>0.2</mu1>
+    <mu2>0.2</mu2>
+  </gazebo>
+  <gazebo reference="wheel3_link">
+    <material>${body_color}</material>
+    <mu1>0.2</mu1>
+    <mu2>0.2</mu2>
+  </gazebo>
+  <gazebo reference="wheel4_link">
+    <material>${body_color}</material>
+    <mu1>0.2</mu1>
+    <mu2>0.2</mu2>
+  </gazebo>
+  <gazebo reference="wheel2_link">
+    <material>${body_color}</material>
+    <mu1>0.2</mu1>
+    <mu2>0.2</mu2>
+  </gazebo>
+  <gazebo reference="wheel1_link">
+    <material>${body_color}</material>
+    <mu1>0.2</mu1>
+    <mu2>0.2</mu2>
+  </gazebo>
+  <gazebo reference="caster_wheel">
+    <material>Gazebo/Grey</material>
+    <mu1>0.2</mu1>
+    <mu2>0.2</mu2>
+  </gazebo>
+  <gazebo reference="caster_axis">
+    <material>Gazebo/Grey</material>
+    <mu1>0.2</mu1>
+    <mu2>0.2</mu2>
+  </gazebo>
   <gazebo reference="lidar_axis">
-        <material>Gazebo/LightGrey</material>
+    <material>Gazebo/LightGrey</material>
   </gazebo>
-<gazebo reference="right_leg">
-  <material>${body_color}</material>
-  <mu1>0.2</mu1>
-  <mu2>0.2</mu2>
-  <selfCollide>true</selfCollide>
-</gazebo>
-<gazebo reference="left_leg">
-  <material>${body_color}</material>
-  <mu1>0.2</mu1>
-  <mu2>0.2</mu2>
-  <selfCollide>true</selfCollide>
-</gazebo>
+  <gazebo reference="right_leg">
+    <material>${body_color}</material>
+    <mu1>0.2</mu1>
+    <mu2>0.2</mu2>
+    <selfCollide>true</selfCollide>
+  </gazebo>
+  <gazebo reference="left_leg">
+    <material>${body_color}</material>
+    <mu1>0.2</mu1>
+    <mu2>0.2</mu2>
+    <selfCollide>true</selfCollide>
+  </gazebo>
+  <gazebo>
+    <plugin name="wheel_drive_controller" filename="libgazebo_ros_diff_drive.so">
+      <ros>
+        <namespace>/diff_drive</namespace>
+      </ros>
+      <!-- wheels -->
+      <num_wheel_pairs>2</num_wheel_pairs>
+      <left_joint>driving1</left_joint>
+      <left_joint>driving4</left_joint>
+      <right_joint>driving2</right_joint>
+      <right_joint>driving3</right_joint>
+      <!-- kinematics -->
+      <wheel_separation>0.4</wheel_separation>
+      <wheel_diameter>0.2</wheel_diameter>
+      <!-- limits -->
+      <max_wheel_torque>20</max_wheel_torque>
+      <max_wheel_acceleration>1.0</max_wheel_acceleration>
+      <!-- output -->
+      <publish_odom>true</publish_odom>
+      <publish_odom_tf>false</publish_odom_tf>
+      <publish_wheel_tf>true</publish_wheel_tf>
+      <odometry_frame>odom</odometry_frame>
+      <robot_base_frame>base_link</robot_base_frame>
+    </plugin>
+  </gazebo>
 </robot>

File: xplore_description/urdf/rover/rover.urdf.xacro (robot description, xacro)
@@ -139,5 +139,5 @@
   </collision>
 </link>
-<link name="wheel2_1ink">
+<link name="wheel2_link">
   <inertial>
     <origin xyz="0.0003394916280188287 -0.010196510227617639 -2.006330920018007e-05" rpy="0 0 0"/>
@@ -159,5 +159,5 @@
   </collision>
 </link>
-<link name="wheel3_1ink">
+<link name="wheel3_link">
   <inertial>
     <origin xyz="0.0003392711202230836 -0.010196510227618527 -1.9767207815879484e-05" rpy="0 0 0"/>
@@ -179,5 +179,5 @@
   </collision>
 </link>
-<link name="wheel1_1ink">
+<link name="wheel1_link">
   <inertial>
     <origin xyz="-0.0003399213580693172 0.010197232694972913 -1.9767207816323573e-05" rpy="0 0 0"/>
@@ -199,5 +199,5 @@
   </collision>
 </link>
-<link name="wheel4_1ink">
+<link name="wheel4_link">
   <inertial>
     <origin xyz="-0.0003391418658636458 0.010197232694973468 -2.0063309200568646e-05" rpy="0 0 0"/>
@@ -350,5 +350,5 @@
   <origin xyz="-0.017133 0.01669 -0.269456" rpy="0 0 0"/>
   <parent link="steering2_link"/>
-  <child link="wheel2_1ink"/>
+  <child link="wheel2_link"/>
   <axis xyz="-0.033267 0.999444 0.002046"/>
 </joint>
@@ -356,5 +356,5 @@
   <origin xyz="-0.017133 0.01669 -0.269457" rpy="0 0 0"/>
   <parent link="steering3_link"/>
-  <child link="wheel3_1ink"/>
+  <child link="wheel3_link"/>
   <axis xyz="-0.033267 0.999444 0.002046"/>
 </joint>
@@ -362,5 +362,5 @@
   <origin xyz="0.017134 -0.016691 -0.269457" rpy="0 0 0"/>
   <parent link="steering1_link"/>
-  <child link="wheel1_1ink"/>
+  <child link="wheel1_link"/>
   <axis xyz="0.033267 -0.999444 0.002046"/>
 </joint>
@@ -368,5 +368,5 @@
   <origin xyz="0.017133 -0.016691 -0.269456" rpy="0 0 0"/>
   <parent link="steering4_link"/>
-  <child link="wheel4_1ink"/>
+  <child link="wheel4_link"/>
   <axis xyz="0.033267 -0.999444 0.002046"/>
 </joint>
