Commit message: feat: improve static cost map

File: xplore_description/urdf/rover/rover.urdf.xacro (robot description, xacro)
@@ -1,37 +1,47 @@
 <?xml version="1.0" ?>
-<robot name="rover" xmlns:xacro="http://www.ros.org/wiki/xacro">
-<xacro:include filename="$(find xplore_description)/urdf/common/materials.xacro" />
-<xacro:include filename="$(find xplore_description)/urdf/rover/rover.transmission.xacro" />
-<xacro:include filename="$(find xplore_description)/urdf/rover/rover.gazebo.xacro" />
-<xacro:include filename="$(find xplore_description)/urdf/rover/lidar/ouster.xacro" />
-<xacro:include filename="$(find xplore_description)/urdf/rover/imu/imu.xacro" />
-<xacro:include filename="$(find xplore_description)/urdf/common/inertial_macro.xacro" />
-<xacro:include filename="$(find xplore_description)/urdf/rover/camera/oakd_camera.xacro" />
-<xacro:include filename="$(find xplore_description)/urdf/rover/rover.ros2_control.xacro" />
-<xacro:property name="rpm_to_Radps" value="${2*pi/60.0}" />     <!-- rotations per minute to Rad per second conversion -->
-<xacro:property name="velocity_scaling" value="1.0" />     <!-- allows to scale all max velocities down at once -->
-<xacro:macro name="aaa_joint_limits" params="lower:=0.0 upper:=0.0 velocity:=${rpm_to_Radps} effort:=100.0">
-  <limit lower="${lower}" upper="${upper}" velocity="${velocity}" effort="${effort}"/>
-</xacro:macro>
-<xacro:property name="joint1_limits">
-  <xacro:aaa_joint_limits lower="${-1.5*pi}" upper="${1.5*pi}" velocity="${3 * rpm_to_Radps * velocity_scaling}" />
-</xacro:property>
-<xacro:property name="joint2_limits">
-  <xacro:aaa_joint_limits lower="${-pi}" upper="${pi/2}" velocity="${1 * rpm_to_Radps * velocity_scaling}" />
-</xacro:property>
-<xacro:property name="joint3_limits">
-  <xacro:aaa_joint_limits lower="${-pi/4}" upper="${pi/4}" velocity="${1.5 * rpm_to_Radps * velocity_scaling}" />
-</xacro:property>
-<xacro:property name="joint4_limits">
-  <xacro:aaa_joint_limits lower="${-2*pi}" upper="${2*pi}" velocity="${6 * rpm_to_Radps * velocity_scaling}" />
-</xacro:property>
-<xacro:property name="joint5_limits">
-  <xacro:aaa_joint_limits lower="${-pi/2}" upper="${pi/2}" velocity="${2 * rpm_to_Radps * velocity_scaling}" />
-</xacro:property>
-<xacro:property name="joint6_limits">
-  <xacro:aaa_joint_limits lower="${-pi}" upper="${pi}" velocity="${6 * rpm_to_Radps * velocity_scaling}" />
-</xacro:property>
-<link name="base_link"></link>
-<joint name="chassis_joint" type="fixed">
+<robot name="rover"
+  xmlns:xacro="http://www.ros.org/wiki/xacro">
+  <xacro:include filename="$(find xplore_description)/urdf/common/materials.xacro" />
+  <xacro:include filename="$(find xplore_description)/urdf/rover/rover.transmission.xacro" />
+  <xacro:include filename="$(find xplore_description)/urdf/rover/rover.gazebo.xacro" />
+  <xacro:include filename="$(find xplore_description)/urdf/rover/lidar/ouster.xacro" />
+  <xacro:include filename="$(find xplore_description)/urdf/rover/imu/imu.xacro" />
+  <xacro:include filename="$(find xplore_description)/urdf/common/inertial_macro.xacro" />
+  <xacro:include filename="$(find xplore_description)/urdf/rover/camera/oakd_camera.xacro" />
+  <xacro:include filename="$(find xplore_description)/urdf/rover/rover.ros2_control.xacro" />
+  <xacro:property name="rpm_to_Radps" value="${2*pi/60.0}" />
+  <!-- rotations per minute to Rad per second conversion -->
+  <xacro:property name="velocity_scaling" value="1.0" />
+  <!-- allows to scale all max velocities down at once -->
+  <xacro:macro name="aaa_joint_limits" params="lower:=0.0 upper:=0.0 velocity:=${rpm_to_Radps} effort:=100.0">
+    <limit lower="${lower}" upper="${upper}" velocity="${velocity}" effort="${effort}"/>
+  </xacro:macro>
+  <xacro:property name="joint1_limits">
+    <xacro:aaa_joint_limits lower="${-1.5*pi}" upper="${1.5*pi}" velocity="${3 * rpm_to_Radps * velocity_scaling}" />
+  </xacro:property>
+  <xacro:property name="joint2_limits">
+    <xacro:aaa_joint_limits lower="${-pi}" upper="${pi/2}" velocity="${1 * rpm_to_Radps * velocity_scaling}" />
+  </xacro:property>
+  <xacro:property name="joint3_limits">
+    <xacro:aaa_joint_limits lower="${-pi/4}" upper="${pi/4}" velocity="${1.5 * rpm_to_Radps * velocity_scaling}" />
+  </xacro:property>
+  <xacro:property name="joint4_limits">
+    <xacro:aaa_joint_limits lower="${-2*pi}" upper="${2*pi}" velocity="${6 * rpm_to_Radps * velocity_scaling}" />
+  </xacro:property>
+  <xacro:property name="joint5_limits">
+    <xacro:aaa_joint_limits lower="${-pi/2}" upper="${pi/2}" velocity="${2 * rpm_to_Radps * velocity_scaling}" />
+  </xacro:property>
+  <xacro:property name="joint6_limits">
+    <xacro:aaa_joint_limits lower="${-pi}" upper="${pi}" velocity="${6 * rpm_to_Radps * velocity_scaling}" />
+  </xacro:property>
+  <link name="base_link"></link>
+  <!-- Robot Footprint -->
+  <link name="base_footprint"/>
+  <joint name="base_joint" type="fixed">
+    <parent link="base_link"/>
+    <child link="base_footprint"/>
+    <origin xyz="0.0 0.0 -0.40" rpy="0 0 0"/>
+  </joint>
+  <joint name="chassis_joint" type="fixed">
     <parent link="base_link"/>
     <child link="chassis_link"/>
@@ -39,231 +49,231 @@
     <axis xyz="0.0 1.0 0.0"/>
   </joint>
-<link name="chassis_link">
-  <inertial>
-    <origin xyz="0.05362398614035063 0.01974617698532859 0.037120813316089823" rpy="0 0 0"/>
-    <mass value="6.257043020156179"/>
-    <inertia ixx="0.340644" iyy="0.466541" izz="0.402706" ixy="0.000337" iyz="0.00055" ixz="-0.092411"/>
-  </inertial>
-  <visual>
-    <origin xyz="0 0 0" rpy="0 0 0"/>
-    <geometry>
-      <mesh filename="file://$(find xplore_description)/meshes/rover/base_link.stl" scale="0.001 0.001 0.001"/>
-    </geometry>
-    <material name="blue"/>
-  </visual>
-  <collision>
-    <origin xyz="0 0 0" rpy="0 0 0"/>
-    <geometry>
-      <mesh filename="file://$(find xplore_description)/meshes/rover/base_link.stl" scale="0.001 0.001 0.001"/>
-    </geometry>
-  </collision>
-</link>
-<link name="steering3_link">
-  <inertial>
-    <origin xyz="-0.01189644601781037 -0.036027929982466456 -0.2129618322901442" rpy="0 0 0"/>
-    <mass value="0.3543584805415501"/>
-    <inertia ixx="0.003558" iyy="0.003121" izz="0.000562" ixy="2e-06" iyz="-0.000206" ixz="-0.000178"/>
-  </inertial>
-  <visual>
-    <origin xyz="-0.421384 -0.393882 0.063562" rpy="0 0 0"/>
-    <geometry>
-      <mesh filename="file://$(find xplore_description)/meshes/rover/steering_1.stl" scale="0.001 0.001 0.001"/>
-    </geometry>
-    <material name="silver"/>
-  </visual>
-  <collision>
-    <origin xyz="-0.421384 -0.393882 0.063562" rpy="0 0 0"/>
-    <geometry>
-      <mesh filename="file://$(find xplore_description)/meshes/rover/steering_1.stl" scale="0.001 0.001 0.001"/>
-    </geometry>
-  </collision>
-</link>
-<link name="steering4_link">
-  <inertial>
-    <origin xyz="0.011896575272170529 0.03602765244982159 -0.21296112839152875" rpy="0 0 0"/>
-    <mass value="0.3543584805415501"/>
-    <inertia ixx="0.003558" iyy="0.003121" izz="0.000562" ixy="2e-06" iyz="0.000206" ixz="0.000178"/>
-  </inertial>
-  <visual>
-    <origin xyz="-0.42341 0.353934 0.012408" rpy="0 0 0"/>
-    <geometry>
-      <mesh filename="file://$(find xplore_description)/meshes/rover/steering_2.stl" scale="0.001 0.001 0.001"/>
-    </geometry>
-    <material name="silver"/>
-  </visual>
-  <collision>
-    <origin xyz="-0.42341 0.353934 0.012408" rpy="0 0 0"/>
-    <geometry>
-      <mesh filename="file://$(find xplore_description)/meshes/rover/steering_2.stl" scale="0.001 0.001 0.001"/>
-    </geometry>
-  </collision>
-</link>
-<link name="steering1_link">
-  <inertial>
-    <origin xyz="0.011896795779964109 0.03602765244982109 -0.21296183229014454" rpy="0 0 0"/>
-    <mass value="0.3543584805415501"/>
-    <inertia ixx="0.003558" iyy="0.003121" izz="0.000562" ixy="2e-06" iyz="0.000206" ixz="0.000178"/>
-  </inertial>
-  <visual>
-    <origin xyz="0.408171 0.353934 0.063562" rpy="0 0 0"/>
-    <geometry>
-      <mesh filename="file://$(find xplore_description)/meshes/rover/steering_3.stl" scale="0.001 0.001 0.001"/>
-    </geometry>
-    <material name="silver"/>
-  </visual>
-  <collision>
-    <origin xyz="0.408171 0.353934 0.063562" rpy="0 0 0"/>
-    <geometry>
-      <mesh filename="file://$(find xplore_description)/meshes/rover/steering_3.stl" scale="0.001 0.001 0.001"/>
-    </geometry>
-  </collision>
-</link>
-<link name="steering2_link">
-  <inertial>
-    <origin xyz="-0.011896225510015512 -0.036027929982466234 -0.21296112839152861" rpy="0 0 0"/>
-    <mass value="0.3543584805415501"/>
-    <inertia ixx="0.003558" iyy="0.003121" izz="0.000562" ixy="2e-06" iyz="-0.000206" ixz="-0.000178"/>
-  </inertial>
-  <visual>
-    <origin xyz="0.410197 -0.393882 0.012408" rpy="0 0 0"/>
-    <geometry>
-      <mesh filename="file://$(find xplore_description)/meshes/rover/steering_4.stl" scale="0.001 0.001 0.001"/>
-    </geometry>
-    <material name="silver"/>
-  </visual>
-  <collision>
-    <origin xyz="0.410197 -0.393882 0.012408" rpy="0 0 0"/>
-    <geometry>
-      <mesh filename="file://$(find xplore_description)/meshes/rover/steering_4.stl" scale="0.001 0.001 0.001"/>
-    </geometry>
-  </collision>
-</link>
-<link name="wheel2_link">
-  <inertial>
-    <origin xyz="0.0003394916280188287 -0.010196510227617639 -2.006330920018007e-05" rpy="0 0 0"/>
-    <mass value="1.592763813314383"/>
-    <inertia ixx="0.010896" iyy="0.018605" izz="0.010887" ixy="-0.000257" iyz="1.6e-05" ixz="-0.0"/>
-  </inertial>
-  <visual>
-    <origin xyz="0.42733 -0.410572 0.281864" rpy="0 0 0"/>
-    <geometry>
-      <mesh filename="file://$(find xplore_description)/meshes/rover/wheel3_1.stl" scale="0.001 0.001 0.001"/>
-    </geometry>
-    <material name="pink"/>
-  </visual>
-  <collision>
-    <origin xyz="0.42733 -0.410572 0.281864" rpy="0 0 0"/>
-    <geometry>
-      <mesh filename="file://$(find xplore_description)/meshes/rover/wheel3_1.stl" scale="0.001 0.001 0.001"/>
-    </geometry>
-  </collision>
-</link>
-<link name="wheel3_link">
-  <inertial>
-    <origin xyz="0.0003392711202230836 -0.010196510227618527 -1.9767207815879484e-05" rpy="0 0 0"/>
-    <mass value="1.592763813314383"/>
-    <inertia ixx="0.010896" iyy="0.018605" izz="0.010887" ixy="-0.000257" iyz="1.6e-05" ixz="-0.0"/>
-  </inertial>
-  <visual>
-    <origin xyz="-0.404251 -0.410572 0.333019" rpy="0 0 0"/>
-    <geometry>
-      <mesh filename="file://$(find xplore_description)/meshes/rover/wheel4_1.stl" scale="0.001 0.001 0.001"/>
-    </geometry>
-    <material name="pink"/>
-  </visual>
-  <collision>
-    <origin xyz="-0.404251 -0.410572 0.333019" rpy="0 0 0"/>
-    <geometry>
-      <mesh filename="file://$(find xplore_description)/meshes/rover/wheel4_1.stl" scale="0.001 0.001 0.001"/>
-    </geometry>
-  </collision>
-</link>
-<link name="wheel1_link">
-  <inertial>
-    <origin xyz="-0.0003399213580693172 0.010197232694972913 -1.9767207816323573e-05" rpy="0 0 0"/>
-    <mass value="1.592763813314383"/>
-    <inertia ixx="0.010896" iyy="0.018605" izz="0.010887" ixy="-0.000257" iyz="-1.6e-05" ixz="0.0"/>
-  </inertial>
-  <visual>
-    <origin xyz="0.391037 0.370625 0.333019" rpy="0 0 0"/>
-    <geometry>
-      <mesh filename="file://$(find xplore_description)/meshes/rover/wheel2_1.stl" scale="0.001 0.001 0.001"/>
-    </geometry>
-    <material name="pink"/>
-  </visual>
-  <collision>
-    <origin xyz="0.391037 0.370625 0.333019" rpy="0 0 0"/>
-    <geometry>
-      <mesh filename="file://$(find xplore_description)/meshes/rover/wheel2_1.stl" scale="0.001 0.001 0.001"/>
-    </geometry>
-  </collision>
-</link>
-<link name="wheel4_link">
-  <inertial>
-    <origin xyz="-0.0003391418658636458 0.010197232694973468 -2.0063309200568646e-05" rpy="0 0 0"/>
-    <mass value="1.592763813314383"/>
-    <inertia ixx="0.010896" iyy="0.018605" izz="0.010887" ixy="-0.000257" iyz="-1.6e-05" ixz="0.0"/>
-  </inertial>
-  <visual>
-    <origin xyz="-0.440543 0.370625 0.281864" rpy="0 0 0"/>
-    <geometry>
-      <mesh filename="file://$(find xplore_description)/meshes/rover/wheel1_1.stl" scale="0.001 0.001 0.001"/>
-    </geometry>
-    <material name="pink"/>
-  </visual>
-  <collision>
-    <origin xyz="-0.440543 0.370625 0.281864" rpy="0 0 0"/>
-    <geometry>
-      <mesh filename="file://$(find xplore_description)/meshes/rover/wheel1_1.stl" scale="0.001 0.001 0.001"/>
-    </geometry>
-  </collision>
-</link>
-<link name="right_leg">
-  <inertial>
-    <origin xyz="0.0009668399350314201 0.11623489359260658 0.013375805290350871" rpy="0 0 0"/>
-    <mass value="1.6615144825592312"/>
-    <inertia ixx="0.007103" iyy="0.220618" izz="0.220639" ixy="-5.6e-05" iyz="-0.000815" ixz="0.013196"/>
-  </inertial>
-  <visual>
-    <origin xyz="-0.006607 -0.250474 0.021516" rpy="0 0 0"/>
-    <geometry>
-      <mesh filename="file://$(find xplore_description)/meshes/rover/pivot_droit_1.stl" scale="0.001 0.001 0.001"/>
-    </geometry>
-    <material name="black"/>
-  </visual>
-  <collision>
-    <origin xyz="-0.006607 -0.250474 0.021516" rpy="0 0 0"/>
-    <geometry>
-      <mesh filename="file://$(find xplore_description)/meshes/rover/pivot_droit_1.stl" scale="0.001 0.001 0.001"/>
-    </geometry>
-  </collision>
-</link>
-<link name="left_leg">
-  <inertial>
-    <origin xyz="-0.0009674901728771402 -0.11623517112525206 0.013375805290350576" rpy="0 0 0"/>
-    <mass value="1.6615144825592312"/>
-    <inertia ixx="0.007103" iyy="0.220618" izz="0.220639" ixy="-5.6e-05" iyz="0.000815" ixz="-0.013196"/>
-  </inertial>
-  <visual>
-    <origin xyz="-0.006607 0.210526 0.021516" rpy="0 0 0"/>
-    <geometry>
-      <mesh filename="file://$(find xplore_description)/meshes/rover/pivot_gauche_1.stl" scale="0.001 0.001 0.001"/>
-    </geometry>
-    <material name="black"/>
-  </visual>
-  <collision>
-    <origin xyz="-0.006607 0.210526 0.021516" rpy="0 0 0"/>
-    <geometry>
-      <mesh filename="file://$(find xplore_description)/meshes/rover/pivot_gauche_1.stl" scale="0.001 0.001 0.001"/>
-    </geometry>
-  </collision>
-</link>
-<joint name="chassis_to_caster_axis" type="continuous">
-  <origin xyz="0.3 0.0 -0.225" rpy="0 -0.6 0"/>
-  <axis xyz="0 0 1"/>
-  <parent link="chassis_link"/>
-  <child link="caster_axis"/>
-</joint>
- <link name="caster_axis">
+  <link name="chassis_link">
+    <inertial>
+      <origin xyz="0.05362398614035063 0.01974617698532859 0.037120813316089823" rpy="0 0 0"/>
+      <mass value="6.257043020156179"/>
+      <inertia ixx="0.340644" iyy="0.466541" izz="0.402706" ixy="0.000337" iyz="0.00055" ixz="-0.092411"/>
+    </inertial>
+    <visual>
+      <origin xyz="0 0 0" rpy="0 0 0"/>
+      <geometry>
+        <mesh filename="file://$(find xplore_description)/meshes/rover/base_link.stl" scale="0.001 0.001 0.001"/>
+      </geometry>
+      <material name="blue"/>
+    </visual>
+    <collision>
+      <origin xyz="0 0 0" rpy="0 0 0"/>
+      <geometry>
+        <mesh filename="file://$(find xplore_description)/meshes/rover/base_link.stl" scale="0.001 0.001 0.001"/>
+      </geometry>
+    </collision>
+  </link>
+  <link name="steering3_link">
+    <inertial>
+      <origin xyz="-0.01189644601781037 -0.036027929982466456 -0.2129618322901442" rpy="0 0 0"/>
+      <mass value="0.3543584805415501"/>
+      <inertia ixx="0.003558" iyy="0.003121" izz="0.000562" ixy="2e-06" iyz="-0.000206" ixz="-0.000178"/>
+    </inertial>
+    <visual>
+      <origin xyz="-0.421384 -0.393882 0.063562" rpy="0 0 0"/>
+      <geometry>
+        <mesh filename="file://$(find xplore_description)/meshes/rover/steering_1.stl" scale="0.001 0.001 0.001"/>
+      </geometry>
+      <material name="silver"/>
+    </visual>
+    <collision>
+      <origin xyz="-0.421384 -0.393882 0.063562" rpy="0 0 0"/>
+      <geometry>
+        <mesh filename="file://$(find xplore_description)/meshes/rover/steering_1.stl" scale="0.001 0.001 0.001"/>
+      </geometry>
+    </collision>
+  </link>
+  <link name="steering4_link">
+    <inertial>
+      <origin xyz="0.011896575272170529 0.03602765244982159 -0.21296112839152875" rpy="0 0 0"/>
+      <mass value="0.3543584805415501"/>
+      <inertia ixx="0.003558" iyy="0.003121" izz="0.000562" ixy="2e-06" iyz="0.000206" ixz="0.000178"/>
+    </inertial>
+    <visual>
+      <origin xyz="-0.42341 0.353934 0.012408" rpy="0 0 0"/>
+      <geometry>
+        <mesh filename="file://$(find xplore_description)/meshes/rover/steering_2.stl" scale="0.001 0.001 0.001"/>
+      </geometry>
+      <material name="silver"/>
+    </visual>
+    <collision>
+      <origin xyz="-0.42341 0.353934 0.012408" rpy="0 0 0"/>
+      <geometry>
+        <mesh filename="file://$(find xplore_description)/meshes/rover/steering_2.stl" scale="0.001 0.001 0.001"/>
+      </geometry>
+    </collision>
+  </link>
+  <link name="steering1_link">
+    <inertial>
+      <origin xyz="0.011896795779964109 0.03602765244982109 -0.21296183229014454" rpy="0 0 0"/>
+      <mass value="0.3543584805415501"/>
+      <inertia ixx="0.003558" iyy="0.003121" izz="0.000562" ixy="2e-06" iyz="0.000206" ixz="0.000178"/>
+    </inertial>
+    <visual>
+      <origin xyz="0.408171 0.353934 0.063562" rpy="0 0 0"/>
+      <geometry>
+        <mesh filename="file://$(find xplore_description)/meshes/rover/steering_3.stl" scale="0.001 0.001 0.001"/>
+      </geometry>
+      <material name="silver"/>
+    </visual>
+    <collision>
+      <origin xyz="0.408171 0.353934 0.063562" rpy="0 0 0"/>
+      <geometry>
+        <mesh filename="file://$(find xplore_description)/meshes/rover/steering_3.stl" scale="0.001 0.001 0.001"/>
+      </geometry>
+    </collision>
+  </link>
+  <link name="steering2_link">
+    <inertial>
+      <origin xyz="-0.011896225510015512 -0.036027929982466234 -0.21296112839152861" rpy="0 0 0"/>
+      <mass value="0.3543584805415501"/>
+      <inertia ixx="0.003558" iyy="0.003121" izz="0.000562" ixy="2e-06" iyz="-0.000206" ixz="-0.000178"/>
+    </inertial>
+    <visual>
+      <origin xyz="0.410197 -0.393882 0.012408" rpy="0 0 0"/>
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