Commit message: fix: fix some typos

File: xplore_description/urdf/rover/rover.gazebo.xacro (robot description, xacro)
@@ -1,4 +1,4 @@
 <?xml version="1.0" ?>
-<robot name="kerby" xmlns:xacro="http://www.ros.org/wiki/xacro" >
+<robot name="rover" xmlns:xacro="http://www.ros.org/wiki/xacro" >
 <xacro:property name="body_color" value="Gazebo/Grey" />
 <gazebo reference="chassis_link">

File: xplore_description/urdf/rover/rover.transmission.xacro (robot description, xacro)
@@ -1,4 +1,4 @@
 <?xml version="1.0" ?>
-<robot name="kerby" xmlns:xacro="http://www.ros.org/wiki/xacro" >
+<robot name="rover" xmlns:xacro="http://www.ros.org/wiki/xacro" >
 <transmission name="steering1_tran">
   <type>transmission_interface/SimpleTransmission</type>
@@ -151,30 +151,30 @@
 //   </actuator>
 // </transmission>
-// <transmission name="R�volution 30_tran">
+// <transmission name="Revolution 30_tran">
 //   <type>transmission_interface/SimpleTransmission</type>
-//   <joint name="R�volution 30">
+//   <joint name="Revolution 30">
 //     <hardwareInterface>hardware_interface/EffortJointInterface</hardwareInterface>
 //   </joint>
-//   <actuator name="R�volution 30_actr">
+//   <actuator name="Revolution 30_actr">
 //     <hardwareInterface>hardware_interface/EffortJointInterface</hardwareInterface>
 //     <mechanicalReduction>1</mechanicalReduction>
 //   </actuator>
 // </transmission>
-// <transmission name="R�volution 31_tran">
+// <transmission name="Revolution 31_tran">
 //   <type>transmission_interface/SimpleTransmission</type>
-//   <joint name="R�volution 31">
+//   <joint name="Revolution 31">
 //     <hardwareInterface>hardware_interface/EffortJointInterface</hardwareInterface>
 //   </joint>
-//   <actuator name="R�volution 31_actr">
+//   <actuator name="Revolution 31_actr">
 //     <hardwareInterface>hardware_interface/EffortJointInterface</hardwareInterface>
 //     <mechanicalReduction>1</mechanicalReduction>
 //   </actuator>
 // </transmission>
-// <transmission name="R�volution 32_tran">
+// <transmission name="Revolution 32_tran">
 //   <type>transmission_interface/SimpleTransmission</type>
-//   <joint name="R�volution 32">
+//   <joint name="Revolution 32">
 //     <hardwareInterface>hardware_interface/EffortJointInterface</hardwareInterface>
 //   </joint>
-//   <actuator name="R�volution 32_actr">
+//   <actuator name="Revolution 32_actr">
 //     <hardwareInterface>hardware_interface/EffortJointInterface</hardwareInterface>
 //     <mechanicalReduction>1</mechanicalReduction>

Commit message: feat: fix controllers bug

File: xplore_description/urdf/rover/rover.gazebo.xacro (robot description, xacro)
@@ -3,9 +3,13 @@
   xmlns:xacro="http://www.ros.org/wiki/xacro">
   <xacro:property name="body_color" value="Gazebo/Grey" />
+  <gazebo>
+    <plugin name="gazebo_ros2_control" filename="libgazebo_ros2_control.so">
+      <parameters>$(find xplore_description)/config/control.yaml</parameters>
+    </plugin>
+  </gazebo>
   <gazebo reference="chassis_link">
     <material>${body_color}</material>
     <mu1>0.2</mu1>
     <mu2>0.2</mu2>
-    <gravity>true</gravity>
   </gazebo>
   <gazebo reference="steering1_link">
@@ -49,14 +53,4 @@
     <mu2>0.2</mu2>
   </gazebo>
-  <gazebo reference="caster_wheel">
-    <material>Gazebo/Grey</material>
-    <mu1>0.2</mu1>
-    <mu2>0.2</mu2>
-  </gazebo>
-  <gazebo reference="caster_axis">
-    <material>Gazebo/Grey</material>
-    <mu1>0.2</mu1>
-    <mu2>0.2</mu2>
-  </gazebo>
   <gazebo reference="lidar_axis">
     <material>Gazebo/LightGrey</material>

File: xplore_description/urdf/rover/rover.ros2_control.xacro (robot description, xacro)
@@ -1,4 +1,4 @@
 <?xml version="1.0"?>
-<robot xmlns:xacro="http://www.ros.org/wiki/xacro">
+<robot name="rover" xmlns:xacro="http://www.ros.org/wiki/xacro">
     <ros2_control name="GazeboSystem" type="system">
         <hardware>
@@ -7,6 +7,6 @@
         <joint name="steering1">
             <command_interface name="position">
-               <param name="min">-3.14</param>
-               <param name="max">3.14</param>
+                <param name="min">-3.14</param>
+                <param name="max">3.14</param>
             </command_interface>
             <state_interface name="position"/>
@@ -16,5 +16,5 @@
             <command_interface name="position">
                 <param name="min">-3.14</param>
-               <param name="max">3.14</param>
+                <param name="max">3.14</param>
             </command_interface>
             <state_interface name="position"/>
@@ -23,6 +23,6 @@
         <joint name="steering3">
             <command_interface name="position">
-              <param name="min">-3.14</param>
-               <param name="max">3.14</param>
+                <param name="min">-3.14</param>
+                <param name="max">3.14</param>
             </command_interface>
             <state_interface name="position"/>
@@ -31,13 +31,13 @@
         <joint name="steering4">
             <command_interface name="position">
-               <param name="min">-3.14</param>
-               <param name="max">3.14</param>
+                <param name="min">-3.14</param>
+                <param name="max">3.14</param>
             </command_interface>
             <state_interface name="position"/>
             <state_interface name="velocity"/>
         </joint>
-      <joint name="driving1">
+        <joint name="driving1">
             <command_interface name="velocity">
-              <param name="min">-10</param>
+                <param name="min">-10</param>
                 <param name="max">10</param>
             </command_interface>
@@ -47,5 +47,5 @@
         <joint name="driving2">
             <command_interface name="velocity">
-               <param name="min">-10</param>
+                <param name="min">-10</param>
                 <param name="max">10</param>
             </command_interface>
@@ -70,21 +70,3 @@
         </joint>
     </ros2_control>
-    <gazebo>
-        <plugin name="gazebo_ros2_control" filename="libgazebo_ros2_control.so">
-            <parameters>$(find xplore_description)/config/control.yaml</parameters>
-        </plugin>
-    </gazebo>
-       <gazebo>
-        <plugin name="rover_joint_state" filename="libgazebo_ros_joint_state_publisher.so">
-            <update_rate>10</update_rate>
-            <joint_name>steering1</joint_name>
-            <joint_name>steering2</joint_name>
-            <joint_name>steering3</joint_name>
-            <joint_name>steering4</joint_name>
-            <joint_name>driving1</joint_name>
-            <joint_name>driving2</joint_name>
-            <joint_name>driving3</joint_name>
-            <joint_name>driving4</joint_name>
-        </plugin>
-    </gazebo>
 </robot>

File: xplore_description/urdf/rover/rover.transmission.xacro (robot description, xacro)
@@ -81,103 +81,3 @@
   </actuator>
 </transmission>
-// <transmission name="joint2_tran">
-//   <type>transmission_interface/SimpleTransmission</type>
-//   <joint name="joint2">
-//     <hardwareInterface>hardware_interface/EffortJointInterface</hardwareInterface>
-//   </joint>
-//   <actuator name="joint2_actr">
-//     <hardwareInterface>hardware_interface/EffortJointInterface</hardwareInterface>
-//     <mechanicalReduction>1</mechanicalReduction>
-//   </actuator>
-// </transmission>
-// <transmission name="joint3_tran">
-//   <type>transmission_interface/SimpleTransmission</type>
-//   <joint name="joint3">
-//     <hardwareInterface>hardware_interface/EffortJointInterface</hardwareInterface>
-//   </joint>
-//   <actuator name="joint3_actr">
-//     <hardwareInterface>hardware_interface/EffortJointInterface</hardwareInterface>
-//     <mechanicalReduction>1</mechanicalReduction>
-//   </actuator>
-// </transmission>
-// <transmission name="joint4_tran">
-//   <type>transmission_interface/SimpleTransmission</type>
-//   <joint name="joint4">
-//     <hardwareInterface>hardware_interface/EffortJointInterface</hardwareInterface>
-//   </joint>
-//   <actuator name="joint4_actr">
-//     <hardwareInterface>hardware_interface/EffortJointInterface</hardwareInterface>
-//     <mechanicalReduction>1</mechanicalReduction>
-//   </actuator>
-// </transmission>
-// <transmission name="joint5_tran">
-//   <type>transmission_interface/SimpleTransmission</type>
-//   <joint name="joint5">
-//     <hardwareInterface>hardware_interface/EffortJointInterface</hardwareInterface>
-//   </joint>
-//   <actuator name="joint5_actr">
-//     <hardwareInterface>hardware_interface/EffortJointInterface</hardwareInterface>
-//     <mechanicalReduction>1</mechanicalReduction>
-//   </actuator>
-// </transmission>
-// <transmission name="joint6_tran">
-//   <type>transmission_interface/SimpleTransmission</type>
-//   <joint name="joint6">
-//     <hardwareInterface>hardware_interface/EffortJointInterface</hardwareInterface>
-//   </joint>
-//   <actuator name="joint6_actr">
-//     <hardwareInterface>hardware_interface/EffortJointInterface</hardwareInterface>
-//     <mechanicalReduction>1</mechanicalReduction>
-//   </actuator>
-// </transmission>
-// <transmission name="finger1_tran">
-//   <type>transmission_interface/SimpleTransmission</type>
-//   <joint name="finger1">
-//     <hardwareInterface>hardware_interface/EffortJointInterface</hardwareInterface>
-//   </joint>
-//   <actuator name="finger1_actr">
-//     <hardwareInterface>hardware_interface/EffortJointInterface</hardwareInterface>
-//     <mechanicalReduction>1</mechanicalReduction>
-//   </actuator>
-// </transmission>
-// <transmission name="finger2_tran">
-//   <type>transmission_interface/SimpleTransmission</type>
-//   <joint name="finger2">
-//     <hardwareInterface>hardware_interface/EffortJointInterface</hardwareInterface>
-//   </joint>
-//   <actuator name="finger2_actr">
-//     <hardwareInterface>hardware_interface/EffortJointInterface</hardwareInterface>
-//     <mechanicalReduction>1</mechanicalReduction>
-//   </actuator>
-// </transmission>
-// <transmission name="Revolution 30_tran">
-//   <type>transmission_interface/SimpleTransmission</type>
-//   <joint name="Revolution 30">
-//     <hardwareInterface>hardware_interface/EffortJointInterface</hardwareInterface>
-//   </joint>
-//   <actuator name="Revolution 30_actr">
-//     <hardwareInterface>hardware_interface/EffortJointInterface</hardwareInterface>
-//     <mechanicalReduction>1</mechanicalReduction>
-//   </actuator>
-// </transmission>
-// <transmission name="Revolution 31_tran">
-//   <type>transmission_interface/SimpleTransmission</type>
-//   <joint name="Revolution 31">
-//     <hardwareInterface>hardware_interface/EffortJointInterface</hardwareInterface>
-//   </joint>
-//   <actuator name="Revolution 31_actr">
-//     <hardwareInterface>hardware_interface/EffortJointInterface</hardwareInterface>
-//     <mechanicalReduction>1</mechanicalReduction>
-//   </actuator>
-// </transmission>
-// <transmission name="Revolution 32_tran">
-//   <type>transmission_interface/SimpleTransmission</type>
-//   <joint name="Revolution 32">
-//     <hardwareInterface>hardware_interface/EffortJointInterface</hardwareInterface>
-//   </joint>
-//   <actuator name="Revolution 32_actr">
-//     <hardwareInterface>hardware_interface/EffortJointInterface</hardwareInterface>
-//     <mechanicalReduction>1</mechanicalReduction>
-//   </actuator>
-// </transmission>
 </robot>

File: xplore_description/urdf/rover/rover.urdf.xacro (robot description, xacro)
@@ -269,47 +269,4 @@
     </collision>
   </link>
-  <joint name="chassis_to_caster_axis" type="continuous">
-    <origin xyz="0.3 0.0 -0.225" rpy="0 -0.6 0"/>
-    <axis xyz="0 0 1"/>
-    <parent link="chassis_link"/>
-    <child link="caster_axis"/>
-  </joint>
-  <link name="caster_axis">
-    <visual>
-      <geometry>
-        <cylinder length="0.45" radius="0.005"/>
-      </geometry>
-    </visual>
-    <collision>
-      <geometry>
-        <cylinder length="0.45" radius="0.005"/>
-      </geometry>
-    </collision>
-    <xacro:inertial_cylinder mass="0.25" length="0.45" radius="0.005">
-      <origin xyz="0 0 0" />
-    </xacro:inertial_cylinder>
-  </link>
-  <joint name="caster_axis_to_caster_wheel" type="continuous">
-    <origin xyz="0 0 -0.25" rpy="${pi/2} 0 0"/>
-    <parent link="caster_axis"/>
-    <axis xyz="0 0 1"/>
-    <child link="caster_wheel"/>
-  </joint>
-  <link name="caster_wheel">
-    <visual>
-      <geometry>
-        <cylinder length="0.05" radius="0.05"/>
-      </geometry>
-    </visual>
-    <collision>
-      <origin xyz="0 0 0" rpy="0 0 0"/>
-      <geometry>
-        <cylinder length="0.05" radius="0.05"/>
-      </geometry>
-    </collision>
-    <xacro:inertial_cylinder mass="0.25" length="0.05" radius="0.05">
-      <origin xyz="0 0 0" />
-    </xacro:inertial_cylinder>
-  </link>
   <joint name="chassis_to_lidar_axis" type="fixed">
     <origin xyz="0.2 0.20 0.12" rpy="0 0 0"/>
@@ -381,5 +338,5 @@
     <axis xyz="0.033267 -0.999444 0.002046"/>
   </joint>
-  <joint name="right_pivot" type="continuous">
+  <joint name="right_pivot" type="fixed">
     <origin xyz="-0.1 0.250474 -0.021516" rpy="0 0 0"/>
     <parent link="chassis_link"/>
@@ -387,5 +344,5 @@
     <axis xyz="0.0 1.0 0.0"/>
   </joint>
-  <joint name="left_pivot" type="continuous">
+  <joint name="left_pivot" type="fixed">
     <origin xyz="-0.1 -0.210526 -0.021516" rpy="0 0 0"/>
     <parent link="chassis_link"/>

File: xplore_description/worlds/marsyard2022.world.xacro (robot description, xacro)
@@ -4,6 +4,8 @@
   <world name="marsyard2022">
     <physics type="ode">
-    <gravity>0 0 -9.81</gravity>
-    <real_time_update_rate>0</real_time_update_rate>
+      <gravity>0 0 -98</gravity>
+      <max_step_size>0.005</max_step_size>
+      <real_time_factor>1</real_time_factor>
+      <real_time_update_rate>1000</real_time_update_rate>
       <ode>
         <solver>

File: xplore_description/worlds/marsyard2023.world.xacro (robot description, xacro)
@@ -3,7 +3,7 @@
 <sdf version="1.7" xmlns:xacro="http://www.ros.org/wiki/xacro">
   <world name="marsyard2023">
-     <gravity>0 0 -9.81</gravity>
+     <gravity>0 0 -98</gravity>
     <physics type="ode">
-      <gravity>0 0 -9.81</gravity>
+      <gravity>0 0 -98</gravity>
       <ode>
         <solver>

Commit message: feat: fix simulation

File: xplore_description/urdf/rover/rover.gazebo.xacro (robot description, xacro)
@@ -13,5 +13,5 @@
       <body_name>base_link</body_name>
       <topic_name>odom</topic_name>
-      <gaussian_noise>0.01</gaussian_noise>
+      <gaussian_noise>0.0</gaussian_noise>
       <frame_name>odom</frame_name>
       <xyz_offset>0 0 0</xyz_offset>
@@ -46,21 +46,21 @@
   <gazebo reference="wheel3_link">
     <material>${body_color}</material>
-    <mu1>0.2</mu1>
-    <mu2>0.2</mu2>
+    <mu1>0.9</mu1>
+    <mu2>0.9</mu2>
   </gazebo>
   <gazebo reference="wheel4_link">
     <material>${body_color}</material>
-    <mu1>0.2</mu1>
-    <mu2>0.2</mu2>
+    <mu1>0.9</mu1>
+    <mu2>0.9</mu2>
   </gazebo>
   <gazebo reference="wheel2_link">
     <material>${body_color}</material>
-    <mu1>0.2</mu1>
-    <mu2>0.2</mu2>
+    <mu1>0.9</mu1>
+    <mu2>0.9</mu2>
   </gazebo>
   <gazebo reference="wheel1_link">
     <material>${body_color}</material>
-    <mu1>0.2</mu1>
-    <mu2>0.2</mu2>
+    <mu1>0.9</mu1>
+    <mu2>0.9</mu2>
   </gazebo>
   <gazebo reference="lidar_axis">

File: xplore_description/urdf/rover/rover.urdf.xacro (robot description, xacro)
@@ -46,5 +46,5 @@
     <parent link="base_link"/>
     <child link="chassis_link"/>
-    <origin xyz="0 0 0 " rpy="0 0 0"/>
+    <origin xyz="0 0 0 " rpy="0 0 3.14"/>
     <axis xyz="0.0 1.0 0.0"/>
   </joint>
