Commit message: feat: link nav2 to sim

File: xplore_description/urdf/rover/imu/imu.xacro (robot description, xacro)
@@ -27,5 +27,5 @@
             <always_on>true</always_on>
             <update_rate>100</update_rate>
-            <visualize>false</visualize>
+            <visualize>true</visualize>
             <pose>0 0 0 0 0 0</pose>
             <plugin name='imu_plugin' filename='libgazebo_ros_imu_sensor.so'>

File: xplore_description/urdf/rover/rover.gazebo.xacro (robot description, xacro)
@@ -6,4 +6,15 @@
     <plugin name="gazebo_ros2_control" filename="libgazebo_ros2_control.so">
       <parameters>$(find xplore_description)/config/control.yaml</parameters>
+    </plugin>
+  </gazebo>
+  <gazebo>
+    <plugin name="p3d_base_controller" filename="libgazebo_ros_p3d.so">
+      <update_rate>100.0</update_rate>
+      <body_name>base_link</body_name>
+      <topic_name>odom</topic_name>
+      <gaussian_noise>0.01</gaussian_noise>
+      <frame_name>map</frame_name>
+      <xyz_offset>0 0 0</xyz_offset>
+      <rpy_offset>0 0 0</rpy_offset>
     </plugin>
   </gazebo>

File: xplore_description/urdf/rover/rover.urdf.xacro (robot description, xacro)
@@ -65,5 +65,5 @@
       <origin xyz="0 0 0" rpy="0 0 0"/>
       <geometry>
-        <mesh filename="file://$(find xplore_description)/meshes/rover/base_link.stl" scale="0.001 0.001 0.001"/>
+        <box size="0.5 0.5 0.1"/>
       </geometry>
     </collision>
@@ -83,7 +83,7 @@
     </visual>
     <collision>
-      <origin xyz="-0.421384 -0.393882 0.063562" rpy="0 0 0"/>
-      <geometry>
-        <mesh filename="file://$(find xplore_description)/meshes/rover/steering_1.stl" scale="0.001 0.001 0.001"/>
+      <origin xyz="0 0 0" rpy="0 0 0"/>
+      <geometry>
+        <cylinder length="0.25" radius="0.005"/>
       </geometry>
     </collision>
@@ -103,7 +103,7 @@
     </visual>
     <collision>
-      <origin xyz="-0.42341 0.353934 0.012408" rpy="0 0 0"/>
-      <geometry>
-        <mesh filename="file://$(find xplore_description)/meshes/rover/steering_2.stl" scale="0.001 0.001 0.001"/>
+      <origin xyz="0 0 0" rpy="0 0 0"/>
+      <geometry>
+        <cylinder length="0.25" radius="0.005"/>
       </geometry>
     </collision>
@@ -123,7 +123,7 @@
     </visual>
     <collision>
-      <origin xyz="0.408171 0.353934 0.063562" rpy="0 0 0"/>
-      <geometry>
-        <mesh filename="file://$(find xplore_description)/meshes/rover/steering_3.stl" scale="0.001 0.001 0.001"/>
+      <origin xyz="0 0 0" rpy="0 0 0"/>
+      <geometry>
+        <cylinder length="0.25" radius="0.005"/>
       </geometry>
     </collision>
@@ -143,7 +143,7 @@
     </visual>
     <collision>
-      <origin xyz="0.410197 -0.393882 0.012408" rpy="0 0 0"/>
-      <geometry>
-        <mesh filename="file://$(find xplore_description)/meshes/rover/steering_4.stl" scale="0.001 0.001 0.001"/>
+      <origin xyz="0 0 0" rpy="0 0 0"/>
+      <geometry>
+        <cylinder length="0.25" radius="0.005"/>
       </geometry>
     </collision>
@@ -163,7 +163,7 @@
     </visual>
     <collision>
-      <origin xyz="0.42733 -0.410572 0.281864" rpy="0 0 0"/>
-      <geometry>
-        <mesh filename="file://$(find xplore_description)/meshes/rover/wheel3_1.stl" scale="0.001 0.001 0.001"/>
+      <origin xyz="0 0 0" rpy="1.57 0 0"/>
+      <geometry>
+        <cylinder length="0.13" radius="0.13"/>
       </geometry>
     </collision>
@@ -183,7 +183,7 @@
     </visual>
     <collision>
-      <origin xyz="-0.404251 -0.410572 0.333019" rpy="0 0 0"/>
-      <geometry>
-        <mesh filename="file://$(find xplore_description)/meshes/rover/wheel4_1.stl" scale="0.001 0.001 0.001"/>
+      <origin xyz="0 0 0" rpy="1.57 0 0"/>
+      <geometry>
+        <cylinder length="0.13" radius="0.13"/>
       </geometry>
     </collision>
@@ -203,7 +203,7 @@
     </visual>
     <collision>
-      <origin xyz="0.391037 0.370625 0.333019" rpy="0 0 0"/>
-      <geometry>
-        <mesh filename="file://$(find xplore_description)/meshes/rover/wheel2_1.stl" scale="0.001 0.001 0.001"/>
+     <origin xyz="0 0 0" rpy="1.57 0 0"/>
+      <geometry>
+        <cylinder length="0.13" radius="0.13"/>
       </geometry>
     </collision>
@@ -223,7 +223,7 @@
     </visual>
     <collision>
-      <origin xyz="-0.440543 0.370625 0.281864" rpy="0 0 0"/>
-      <geometry>
-        <mesh filename="file://$(find xplore_description)/meshes/rover/wheel1_1.stl" scale="0.001 0.001 0.001"/>
+      <origin xyz="0 0 0" rpy="1.57 0 0"/>
+      <geometry>
+        <cylinder length="0.13" radius="0.13"/>
       </geometry>
     </collision>
@@ -243,7 +243,7 @@
     </visual>
     <collision>
-      <origin xyz="-0.006607 -0.250474 0.021516" rpy="0 0 0"/>
-      <geometry>
-        <mesh filename="file://$(find xplore_description)/meshes/rover/pivot_droit_1.stl" scale="0.001 0.001 0.001"/>
+      <origin xyz="0 0.1 0" rpy="0 0 0"/>
+      <geometry>
+        <box size="0.8 0.2 0.1"/>
       </geometry>
     </collision>
@@ -263,7 +263,7 @@
     </visual>
     <collision>
-      <origin xyz="-0.006607 0.210526 0.021516" rpy="0 0 0"/>
-      <geometry>
-        <mesh filename="file://$(find xplore_description)/meshes/rover/pivot_gauche_1.stl" scale="0.001 0.001 0.001"/>
+      <origin xyz="0 -0.1 0" rpy="0 0 0"/>
+      <geometry>
+        <box size="0.8 0.2 0.1"/>
       </geometry>
     </collision>
@@ -338,5 +338,48 @@
     <axis xyz="0.033267 -0.999444 0.002046"/>
   </joint>
-  <joint name="right_pivot" type="fixed">
+  <joint name="chassis_to_caster_axis" type="continuous">
+    <origin xyz="0.3 0.0 -0.225" rpy="0 -0.6 0"/>
+    <axis xyz="0 0 1"/>
+    <parent link="chassis_link"/>
+    <child link="caster_axis"/>
+  </joint>
+  <link name="caster_axis">
+    <visual>
+      <geometry>
+        <cylinder length="0.45" radius="0.005"/>
+      </geometry>
+    </visual>
+    <collision>
+      <geometry>
+        <cylinder length="0.45" radius="0.005"/>
+      </geometry>
+    </collision>
+    <xacro:inertial_cylinder mass="0.25" length="0.45" radius="0.005">
+      <origin xyz="0 0 0" />
+    </xacro:inertial_cylinder>
+  </link>
+  <joint name="caster_axis_to_caster_wheel" type="continuous">
+    <origin xyz="0 0 -0.25" rpy="${pi/2} 0 0"/>
+    <parent link="caster_axis"/>
+    <axis xyz="0 0 1"/>
+    <child link="caster_wheel"/>
+  </joint>
+  <link name="caster_wheel">
+    <visual>
+      <geometry>
+        <cylinder length="0.05" radius="0.05"/>
+      </geometry>
+    </visual>
+    <collision>
+      <origin xyz="0 0 0" rpy="0 0 0"/>
+      <geometry>
+        <cylinder length="0.05" radius="0.05"/>
+      </geometry>
+    </collision>
+    <xacro:inertial_cylinder mass="0.25" length="0.05" radius="0.05">
+      <origin xyz="0 0 0" />
+    </xacro:inertial_cylinder>
+  </link>
+  <joint name="right_pivot" type="continuous">
     <origin xyz="-0.1 0.250474 -0.021516" rpy="0 0 0"/>
     <parent link="chassis_link"/>
@@ -344,5 +387,5 @@
     <axis xyz="0.0 1.0 0.0"/>
   </joint>
-  <joint name="left_pivot" type="fixed">
+  <joint name="left_pivot" type="continuous">
     <origin xyz="-0.1 -0.210526 -0.021516" rpy="0 0 0"/>
     <parent link="chassis_link"/>

File: xplore_description/worlds/marsyard2022.world.xacro (robot description, xacro)
@@ -4,6 +4,6 @@
   <world name="marsyard2022">
     <physics type="ode">
-      <gravity>0 0 -98</gravity>
-      <max_step_size>0.005</max_step_size>
+      <gravity>0 0 -9.8</gravity>
+      <max_step_size>0.001</max_step_size>
       <real_time_factor>1</real_time_factor>
       <real_time_update_rate>1000</real_time_update_rate>

File: xplore_description/worlds/marsyard2023.world.xacro (robot description, xacro)
@@ -3,7 +3,7 @@
 <sdf version="1.7" xmlns:xacro="http://www.ros.org/wiki/xacro">
   <world name="marsyard2023">
-     <gravity>0 0 -98</gravity>
+     <gravity>0 0 -9.8</gravity>
     <physics type="ode">
-      <gravity>0 0 -98</gravity>
+      <gravity>0 0 -9.8</gravity>
       <ode>
         <solver>
